File: Duiventrack v1.sch (KiCad schematic (older format))
At the start: 21 parts, among them P1 CONN_01X06, U1 MCP1711-SOT23-5, U2 SP-ABZ-G

Commit message: Aanpassingen gemaakt samen met Remy, board ontwerp
Parts:
- removed JP1: Jumper_NO_Small, Footprint:SolderJumper_NO, symbol Jumper_NO_Small
- removed P1: CONN_01X06, Pin_Headers:Pin_Header_Straight_1x06_Pitch1.27mm, symbol CONN_01X06
- added C10: F, Capacitors_SMD:C_0402, symbol C
- added C11: 1uF, Capacitors_SMD:C_0402, symbol C
- added L1: L, Inductors_SMD:L_0402, symbol L
- added P1: CONN_01X07, Pin_Headers:Pin_Header_Straight_1x07_Pitch1.27mm_SMD_Pin1Right, symbol CONN_01X07
- added P2: CONN_01X02, Pin_Headers:Pin_Header_Straight_1x02_Pitch1.27mm, symbol CONN_01X02
- added R6: 100K, Resistors_SMD:R_0402, symbol R
- C3, C4: footprint Capacitors_SMD:C_0402 -> Capacitors_SMD:C_0603
- C8: value 2.2pF -> F
Connections:
- net +3V3: now also C11.1
- net Earth: now also C10.2, C11.2, P1.7 (P7)
- net MCU_RST: now also P1.2 (P2)
- net SWCLK: now also P1.3 (P3)
- net SWDIO: now also P1.4 (P4)
- net Uart_RX: now also P1.5 (P5)
- net Uart_TX: now also P1.6 (P6)
- net Vbat: now also P1.1 (P1), R6.2
- net at AE1.1 (A), C8.1: now also L1.2; no longer U2.26 (ANT)
- net at R3.2, U1.3 (~SHDN): now also P2.2 (P2)
- new net: C10.1, L1.1, U2.26 (ANT)
- new net: P2.1 (P1), R6.1
Other:
- moved on the sheet: C8, R3
Changed lines of the file:
@@
 F 0 "C3" H 6025 2050 50  0000 L CNN
 F 1 "10uF" H 6025 1850 50  0000 L CNN
-F 2 "Capacitors_SMD:C_0402" H 6038 1800 50  0001 C CNN
+F 2 "Capacitors_SMD:C_0603" H 6038 1800 50  0001 C CNN
 F 3 "" H 6000 1950 50  0000 C CNN
 	1    6000 1950
@@
 F 0 "C4" H 6375 1400 50  0000 L CNN
 F 1 "10uF" H 6375 1200 50  0000 L CNN
-F 2 "Capacitors_SMD:C_0402" H 6388 1150 50  0001 C CNN
+F 2 "Capacitors_SMD:C_0603" H 6388 1150 50  0001 C CNN
 F 3 "" H 6350 1300 50  0000 C CNN
 	1    6350 1300
@@
 	1    0    0    -1
 $EndComp
-$Comp
-L Jumper_NO_Small JP1
-U 1 1 5AD79D47
-P 2400 2200
-F 0 "JP1" H 2400 2280 50  0000 C CNN
-F 1 "Jumper_NO_Small" H 2410 2140 50  0000 C CNN
-F 2 "Footprint:SolderJumper_NO" H 2400 2200 50  0001 C CNN
-F 3 "" H 2400 2200 50  0000 C CNN
-	1    2400 2200
-	1    0    0    -1
-$EndComp
 Wire Wire Line
 	7050 1750 5800 1750
@@
 Wire Wire Line
 	6650 3950 6650 3800
-Wire Wire Line
-	8050 3950 6650 3950
 Wire Wire Line
 	3250 3100 3250 3050
@@
 	2950 3500 3600 3500
 Wire Wire Line
-	3250 3400 3250 4000
-Wire Wire Line
-	3250 4000 3750 4000
+	3250 3400 3250 4100
 Connection ~ 3250 3500
 Wire Wire Line
@@
 L Earth #PWR015
 U 1 1 5AD80891
-P 3700 4600
-F 0 "#PWR015" H 3700 4350 50  0001 C CNN
-F 1 "Earth" H 3700 4450 50  0001 C CNN
-F 2 "" H 3700 4600 50  0000 C CNN
-F 3 "" H 3700 4600 50  0000 C CNN
-	1    3700 4600
-	1    0    0    -1
-$EndComp
-Wire Wire Line
-	3750 4500 3700 4500
-Wire Wire Line
-	3700 4500 3700 4600
+P 3950 4600
+F 0 "#PWR015" H 3950 4350 50  0001 C CNN
+F 1 "Earth" H 3950 4450 50  0001 C CNN
+F 2 "" H 3950 4600 50  0000 C CNN
+F 3 "" H 3950 4600 50  0000 C CNN
+	1    3950 4600
+	1    0    0    -1
+$EndComp
 Text GLabel 8000 3750 0    39   Input ~ 0
 SWDIO
@@
 Wire Wire Line
 	8000 3750 8050 3750
-Text GLabel 3700 4100 0    39   Input ~ 0
+Text GLabel 3950 4200 0    39   Input ~ 0
 SWCLK
-Text GLabel 3700 4200 0    39   Input ~ 0
+Text GLabel 3950 4300 0    39   Input ~ 0
 SWDIO
-Wire Wire Line
-	3700 4100 3750 4100
-Wire Wire Line
-	3700 4200 3750 4200
-$Comp
-L CONN_01X06 P1
-U 1 1 5AD822F9
-P 3950 4250
-F 0 "P1" H 3950 4600 50  0000 C CNN
-F 1 "CONN_01X06" V 4050 4250 50  0000 C CNN
-F 2 "Pin_Headers:Pin_Header_Straight_1x06_Pitch1.27mm" H 3950 4250 50  0001 C CNN
-F 3 "" H 3950 4250 50  0000 C CNN
-	1    3950 4250
-	1    0    0    -1
-$EndComp
 Text GLabel 10300 2350 2    39   Input ~ 0
 Uart_TX
@@
 Wire Wire Line
 	10250 2250 10300 2250
-Text GLabel 3700 4300 0    39   Input ~ 0
+Text GLabel 3950 4400 0    39   Input ~ 0
 Uart_RX
-Text GLabel 3700 4400 0    39   Input ~ 0
+Text GLabel 3950 4500 0    39   Input ~ 0
 Uart_TX
-Wire Wire Line
-	3700 4300 3750 4300
-Wire Wire Line
-	3700 4400 3750 4400
 NoConn ~ 10250 1350
 NoConn ~ 10250 1500
@@
 L C C8
 U 1 1 5AE853A6
-P 7150 4200
-F 0 "C8" H 7175 4300 50  0000 L CNN
-F 1 "2.2pF" H 7175 4100 50  0000 L CNN
-F 2 "Capacitors_SMD:C_0402" H 7188 4050 50  0001 C CNN
-F 3 "" H 7150 4200 50  0000 C CNN
-	1    7150 4200
+P 7000 4200
+F 0 "C8" H 7025 4300 50  0000 L CNN
+F 1 "F" H 7025 4100 50  0000 L CNN
+F 2 "Capacitors_SMD:C_0402" H 7038 4050 50  0001 C CNN
+F 3 "" H 7000 4200 50  0000 C CNN
+	1    7000 4200
 	1    0    0    -1
 $EndComp
@@
 L Earth #PWR016
 U 1 1 5AE85758
-P 7150 4350
-F 0 "#PWR016" H 7150 4100 50  0001 C CNN
-F 1 "Earth" H 7150 4200 50  0001 C CNN
-F 2 "" H 7150 4350 50  0000 C CNN
-F 3 "" H 7150 4350 50  0000 C CNN
-	1    7150 4350
-	1    0    0    -1
-$EndComp
-Wire Wire Line
-	7150 4050 7150 3950
-Connection ~ 7150 3950
+P 7000 4350
+F 0 "#PWR016" H 7000 4100 50  0001 C CNN
+F 1 "Earth" H 7000 4200 50  0001 C CNN
+F 2 "" H 7000 4350 50  0000 C CNN
+F 3 "" H 7000 4350 50  0000 C CNN
+	1    7000 4350
+	1    0    0    -1
+$EndComp
 $Comp
 L SP-ABZ-G U2
@@
 L R R3
 U 1 1 5AE86CF1
-P 2550 2500
-F 0 "R3" V 2630 2500 50  0000 C CNN
-F 1 "1M" V 2550 2500 50  0000 C CNN
-F 2 "Resistors_SMD:R_0402" V 2480 2500 50  0001 C CNN
-F 3 "" H 2550 2500 50  0000 C CNN
-	1    2550 2500
+P 2600 2750
+F 0 "R3" V 2680 2750 50  0000 C CNN
+F 1 "1M" V 2600 2750 50  0000 C CNN
+F 2 "Resistors_SMD:R_0402" V 2530 2750 50  0001 C CNN
+F 3 "" H 2600 2750 50  0000 C CNN
+	1    2600 2750
 	-1   0    0    1
 $EndComp
@@
 L Earth #PWR017
 U 1 1 5AE87323
-P 2550 2700
-F 0 "#PWR017" H 2550 2450 50  0001 C CNN
-F 1 "Earth" H 2550 2550 50  0001 C CNN
-F 2 "" H 2550 2700 50  0000 C CNN
-F 3 "" H 2550 2700 50  0000 C CNN
-	1    2550 2700
-	1    0    0    -1
-$EndComp
-Wire Wire Line
-	2450 1850 2450 1950
-Wire Wire Line
-	2450 1950 2550 1950
-Wire Wire Line
-	2550 1950 2550 2350
-Wire Wire Line
-	2550 2200 2500 2200
-Wire Wire Line
-	2550 2650 2550 2700
-Connection ~ 2550 2200
-Wire Wire Line
-	2300 2200 2250 2200
-Wire Wire Line
-	2250 2200 2250 1450
-Connection ~ 2250 1450
+P 2600 2950
+F 0 "#PWR017" H 2600 2700 50  0001 C CNN
+F 1 "Earth" H 2600 2800 50  0001 C CNN
+F 2 "" H 2600 2950 50  0000 C CNN
+F 3 "" H 2600 2950 50  0000 C CNN
+	1    2600 2950
+	1    0    0    -1
+$EndComp
+Wire Wire Line
+	2450 1850 2450 2100
+Wire Wire Line
+	2600 2900 2600 2950
+Wire Wire Line
+	2300 2450 2950 2450
 NoConn ~ 8050 1900
+$Comp
+L R R6
+U 1 1 5AEC2243
+P 2300 2150
+F 0 "R6" V 2380 2150 50  0000 C CNN
+F 1 "100K" V 2300 2150 50  0000 C CNN
+F 2 "Resistors_SMD:R_0402" V 2230 2150 50  0001 C CNN
+F 3 "" H 2300 2150 50  0000 C CNN
+	1    2300 2150
+	-1   0    0    1
+$EndComp
+Wire Wire Line
+	2300 2000 2300 1450
+Connection ~ 2300 1450
+Wire Wire Line
+	2300 2450 2300 2300
+Wire Wire Line
+	2600 2100 2600 2600
+Wire Wire Line
+	2450 2100 2600 2100
+$Comp
+L CONN_01X02 P2
+U 1 1 5AEC3055
+P 3150 2500
+F 0 "P2" H 3150 2650 50  0000 C CNN
+F 1 "CONN_01X02" V 3250 2500 50  0000 C CNN
+F 2 "Pin_Headers:Pin_Header_Straight_1x02_Pitch1.27mm" H 3150 2500 50  0001 C CNN
+F 3 "" H 3150 2500 50  0000 C CNN
+	1    3150 2500
+	1    0    0    -1
+$EndComp
+Wire Wire Line
+	2950 2550 2600 2550
+Connection ~ 2600 2550
+$Comp
+L C C10
+U 1 1 5AEC3DC6
+P 7500 4200
+F 0 "C10" H 7525 4300 50  0000 L CNN
+F 1 "F" H 7525 4100 50  0000 L CNN
+F 2 "Capacitors_SMD:C_0402" H 7538 4050 50  0001 C CNN
+F 3 "" H 7500 4200 50  0000 C CNN
+	1    7500 4200
+	1    0    0    -1
+$EndComp
+$Comp
+L Earth #PWR018
+U 1 1 5AEC3F45
+P 7500 4350
+F 0 "#PWR018" H 7500 4100 50  0001 C CNN
+F 1 "Earth" H 7500 4200 50  0001 C CNN
+F 2 "" H 7500 4350 50  0000 C CNN
+F 3 "" H 7500 4350 50  0000 C CNN
+	1    7500 4350
+	1    0    0    -1
+$EndComp
+Wire Wire Line
+	7500 4050 7500 3950
+Connection ~ 7500 3950
+$Comp
+L L L1
+U 1 1 5AEC4077
+P 7250 3950
+F 0 "L1" V 7200 3950 50  0000 C CNN
+F 1 "L" V 7325 3950 50  0000 C CNN
+F 2 "Inductors_SMD:L_0402" H 7250 3950 50  0001 C CNN
+F 3 "" H 7250 3950 50  0000 C CNN
+	1    7250 3950
+	0    1    1    0
+$EndComp
+Wire Wire Line
+	8050 3950 7400 3950
+Wire Wire Line
+	7100 3950 6650 3950
+Wire Wire Line
+	7000 4050 7000 3950
+Connection ~ 7000 3950
+$Comp
+L CONN_01X07 P1
+U 1 1 5AEC3D1A
+P 4150 4300
+F 0 "P1" H 4150 4700 50  0000 C CNN
+F 1 "CONN_01X07" V 4250 4300 50  0000 C CNN
+F 2 "Pin_Headers:Pin_Header_Straight_1x07_Pitch1.27mm_SMD_Pin1Right" H 4150 4300 50  0001 C CNN
+F 3 "" H 4150 4300 50  0000 C CNN
+	1    4150 4300
+	1    0    0    -1
+$EndComp
+Text GLabel 3950 4000 0    39   Input ~ 0
+Vbat
+Wire Wire Line
+	3250 4100 3950 4100
+$Comp
+L C C11
+U 1 1 5AECCB73
+P 3700 1700
+F 0 "C11" H 3725 1800 50  0000 L CNN
+F 1 "1uF" H 3725 1600 50  0000 L CNN
+F 2 "Capacitors_SMD:C_0402" H 3738 1550 50  0001 C CNN
+F 3 "" H 3700 1700 50  0000 C CNN
+	1    3700 1700
+	1    0    0    -1
+$EndComp
+$Comp
+L Earth #PWR019
+U 1 1 5AECCC49
+P 3700 1850
+F 0 "#PWR019" H 3700 1600 50  0001 C CNN
+F 1 "Earth" H 3700 1700 50  0001 C CNN
+F 2 "" H 3700 1850 50  0000 C CNN
+F 3 "" H 3700 1850 50  0000 C CNN
+	1    3700 1850
+	1    0    0    -1
+$EndComp
+Wire Wire Line
+	3700 1550 3700 1450
+Connection ~ 3700 1450
 $EndSCHEMATC

Commit message: Aanpassingen gemaakt aan het board, vooral de achterzijde, connector is anders aangesloten
Connections:
- net MCU_RST: now also P1.6 (P6); no longer P1.2 (P2)
- net SWCLK: now also P1.2 (P2); no longer P1.3 (P3)
- net SWDIO: now also P1.3 (P3); no longer P1.4 (P4)
- net Uart_RX: now also P1.4 (P4); no longer P1.5 (P5)
- net Uart_TX: now also P1.5 (P5); no longer P1.6 (P6)
Changed lines of the file:
@@
 	2950 3500 3600 3500
 Wire Wire Line
-	3250 3400 3250 4100
+	3250 3400 3250 4500
 Connection ~ 3250 3500
 Wire Wire Line
@@
 Wire Wire Line
 	8000 3750 8050 3750
+Text GLabel 3950 4100 0    39   Input ~ 0
+SWCLK
 Text GLabel 3950 4200 0    39   Input ~ 0
-SWCLK
-Text GLabel 3950 4300 0    39   Input ~ 0
 SWDIO
 Text GLabel 10300 2350 2    39   Input ~ 0
@@
 Wire Wire Line
 	10250 2250 10300 2250
+Text GLabel 3950 4300 0    39   Input ~ 0
+Uart_RX
 Text GLabel 3950 4400 0    39   Input ~ 0
-Uart_RX
-Text GLabel 3950 4500 0    39   Input ~ 0
 Uart_TX
 NoConn ~ 10250 1350
@@
 Text GLabel 3950 4000 0    39   Input ~ 0
 Vbat
-Wire Wire Line
-	3250 4100 3950 4100
 $Comp
 L C C11
@@
 	3700 1550 3700 1450
 Connection ~ 3700 1450
+Wire Wire Line
+	3250 4500 3950 4500
 $EndSCHEMATC

Commit message: Crystal toegevoegd
Parts:
- added C12, C13: 20pF, Capacitors_SMD:C_0402, symbol C
- added Y1: Crystal, Crystals:Crystal_SMD_5032-2pin_5.0x3.2mm, symbol Crystal
Connections:
- net +3V3: no longer U2.48 (VDD_TCXO)
- net Earth: now also C12.2, C13.2
- net PA12: now reaches U2.1 (PA12/USB_DP)
- net PA12: now also U2.48 (VDD_TCXO)
- net at U2.45 (PH1-OSC_OUT): now also C12.1, Y1.1
- net at U2.46 (PH0-OSC_IN): now also C13.1, Y1.2
- no-connect marks 31 -> 28
Other:
- moved on the sheet: C2, C9, P1, R1, R2, R4, R5, TP1

Commit message: Revert "Crystal toegevoegd"
This reverts commit 51f246dfdab6a70a9bd41b0f28c72966c573f5f4.
Parts:
- removed C12, C13: 20pF, Capacitors_SMD:C_0402, symbol C
- removed Y1: Crystal, Crystals:Crystal_SMD_5032-2pin_5.0x3.2mm, symbol Crystal
Connections:
- net +3V3: now also U2.48 (VDD_TCXO)
- net PA12: no longer names the net of U2.1 (PA12/USB_DP)
- net PA12: no longer U2.48 (VDD_TCXO)
- no-connect marks 28 -> 31
Other:
- moved on the sheet: C2, C9, P1, R1, R2, R4, R5, TP1
