File: Duiventrack v1.sch (KiCad schematic (older format))
At the start: 28 parts, among them P1 CONN_01X07, P2 CONN_01X02, U1 MCP1711-SOT23-5, U2 SP-ABZ-G

Commit message: Via en SolderJumper toegevoegd
Parts:
- JP2: footprint (none) -> Footprint:SolderJumper_NO-3
Changed lines of the file:
@@
 F 0 "JP2" H 7950 850 50  0000 L CNN
 F 1 "Jumper_NC_Dual" H 7900 1050 50  0000 C BNN
-F 2 "" H 7900 950 50  0001 C CNN
+F 2 "Footprint:SolderJumper_NO-3" H 7900 950 50  0001 C CNN
 F 3 "" H 7900 950 50  0000 C CNN
 	1    7900 950
