File: Duiventrack v1.kicad_pcb (KiCad board)
At the start: 2 copper layers, 22.6 x 12.8 mm, 28 parts, among them P1 CONN_01X07, P2 CONN_01X02, U1 MCP1711-SOT23-5, U2 SP-ABZ-G

Commit message: Small changes
Parts:
- moved R1 2.20 mm to (151.1, 96.8), turned to 0 degrees
- moved C1 0.90 mm to (145.8, 87.1)
- moved R2 0.84 mm to (153.0, 96.5)
Routing:
- net VBat: track 33.0 -> 29.4 mm
- net VBat_Measure: track 3.47 -> 4.43 mm
Changed lines of the file:
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@@
-(kicad_pcb (version 4) (host pcbnew 4.0.5)
+(kicad_pcb (version 4) (host pcbnew 4.0.6)
   (general
     (links 74)
-    (no_connects 13)
+    (no_connects 9)
     (area 139.724999 84.924999 162.475001 97.875001)
     (thickness 1.6)
     (drawings 10)
-    (tracks 175)
+    (tracks 174)
     (zones 0)
     (modules 28)
@@
     (add_net VBat_Measure)
   )
-  (module Resistors_SMD:R_0402 (layer B.Cu)
-    (at 141.25 91.6)
-    (descr "Resistor SMD 0402, reflow soldering, Vishay (see dcrcw.pdf)")
-    (tags "resistor 0402")
-    (attr smd)
-    (fp_text reference R3 (at -1.15 0 270) (layer B.SilkS)
-      (effects (font (size 0.5 0.5) (thickness 0.08)) (justify mirror))
-    )
-    (fp_text value 1M (at 0 -1.45) (layer B.Fab)
-      (effects (font (size 1 1) (thickness 0.15)) (justify mirror))
-    )
-    (fp_text user %R (at 0 1.35) (layer B.Fab)
-      (effects (font (size 1 1) (thickness 0.15)) (justify mirror))
-    )
-    (fp_line (start -0.5 -0.25) (end -0.5 0.25) (layer B.Fab) (width 0.1))
-    (fp_line (start 0.5 -0.25) (end -0.5 -0.25) (layer B.Fab) (width 0.1))
-    (fp_line (start 0.5 0.25) (end 0.5 -0.25) (layer B.Fab) (width 0.1))
-    (fp_line (start -0.5 0.25) (end 0.5 0.25) (layer B.Fab) (width 0.1))
-    (fp_line (start 0.25 0.53) (end -0.25 0.53) (layer B.SilkS) (width 0.12))
-    (fp_line (start -0.25 -0.53) (end 0.25 -0.53) (layer B.SilkS) (width 0.12))
-    (fp_line (start -0.8 0.45) (end 0.8 0.45) (layer B.CrtYd) (width 0.05))
-    (fp_line (start -0.8 0.45) (end -0.8 -0.45) (layer B.CrtYd) (width 0.05))
-    (fp_line (start 0.8 -0.45) (end 0.8 0.45) (layer B.CrtYd) (width 0.05))
-    (fp_line (start 0.8 -0.45) (end -0.8 -0.45) (layer B.CrtYd) (width 0.05))
-    (pad 1 smd rect (at -0.45 0) (size 0.4 0.6) (layers B.Cu B.Paste B.Mask)
-      (net 2 Earth))
-    (pad 2 smd rect (at 0.45 0) (size 0.4 0.6) (layers B.Cu B.Paste B.Mask)
-      (net 14 "Net-(P2-Pad2)"))
-    (model ${KISYS3DMOD}/Resistors_SMD.3dshapes/R_0402.wrl
-      (at (xyz 0 0 0))
-      (scale (xyz 1 1 1))
-      (rotate (xyz 0 0 0))
-    )
-  )
   (module Footprint:Murata_SP-ABZ-G (layer F.Cu)
     (at 149.85 91.35)
@@
       (scale (xyz 0.39 0.39 0.39))
       (rotate (xyz 90 0 180))
+    )
+  )
+  (module Resistors_SMD:R_0402 (layer B.Cu)
+    (at 141.25 91.6)
+    (descr "Resistor SMD 0402, reflow soldering, Vishay (see dcrcw.pdf)")
+    (tags "resistor 0402")
+    (attr smd)
+    (fp_text reference R3 (at -1.15 0 270) (layer B.SilkS)
+      (effects (font (size 0.5 0.5) (thickness 0.08)) (justify mirror))
+    )
+    (fp_text value 1M (at 0 -1.45) (layer B.Fab)
+      (effects (font (size 1 1) (thickness 0.15)) (justify mirror))
+    )
+    (fp_text user %R (at 0 1.35) (layer B.Fab)
+      (effects (font (size 1 1) (thickness 0.15)) (justify mirror))
+    )
+    (fp_line (start -0.5 -0.25) (end -0.5 0.25) (layer B.Fab) (width 0.1))
+    (fp_line (start 0.5 -0.25) (end -0.5 -0.25) (layer B.Fab) (width 0.1))
+    (fp_line (start 0.5 0.25) (end 0.5 -0.25) (layer B.Fab) (width 0.1))
+    (fp_line (start -0.5 0.25) (end 0.5 0.25) (layer B.Fab) (width 0.1))
+    (fp_line (start 0.25 0.53) (end -0.25 0.53) (layer B.SilkS) (width 0.12))
+    (fp_line (start -0.25 -0.53) (end 0.25 -0.53) (layer B.SilkS) (width 0.12))
+    (fp_line (start -0.8 0.45) (end 0.8 0.45) (layer B.CrtYd) (width 0.05))
+    (fp_line (start -0.8 0.45) (end -0.8 -0.45) (layer B.CrtYd) (width 0.05))
+    (fp_line (start 0.8 -0.45) (end 0.8 0.45) (layer B.CrtYd) (width 0.05))
+    (fp_line (start 0.8 -0.45) (end -0.8 -0.45) (layer B.CrtYd) (width 0.05))
+    (pad 1 smd rect (at -0.45 0) (size 0.4 0.6) (layers B.Cu B.Paste B.Mask)
+      (net 2 Earth))
+    (pad 2 smd rect (at 0.45 0) (size 0.4 0.6) (layers B.Cu B.Paste B.Mask)
+      (net 14 "Net-(P2-Pad2)"))
+    (model ${KISYS3DMOD}/Resistors_SMD.3dshapes/R_0402.wrl
+      (at (xyz 0 0 0))
+      (scale (xyz 1 1 1))
+      (rotate (xyz 0 0 0))
     )
   )
@@
   )
   (module Capacitors_SMD:C_0402 (layer B.Cu)
-    (at 146 86.25 270)
+    (at 145.796 87.122 270)
     (descr "Capacitor SMD 0402, reflow soldering, AVX (see smccp.pdf)")
     (tags "capacitor 0402")
@@
   )
   (module Resistors_SMD:R_0402 (layer B.Cu)
-    (at 153.3 96.4 90)
+    (at 151.13 96.774)
     (descr "Resistor SMD 0402, reflow soldering, Vishay (see dcrcw.pdf)")
     (tags "resistor 0402")
     (attr smd)
-    (fp_text reference R1 (at 1.2 0 180) (layer B.SilkS)
+    (fp_text reference R1 (at 1.2 0 90) (layer B.SilkS)
       (effects (font (size 0.5 0.5) (thickness 0.08)) (justify mirror))
     )
-    (fp_text value 10M (at 0 -1.45 90) (layer B.Fab)
-      (effects (font (size 1 1) (thickness 0.15)) (justify mirror))
-    )
-    (fp_text user %R (at 0 1.35 90) (layer B.Fab)
+    (fp_text value 10M (at 0 -1.45) (layer B.Fab)
+      (effects (font (size 1 1) (thickness 0.15)) (justify mirror))
+    )
+    (fp_text user %R (at 0 1.35) (layer B.Fab)
       (effects (font (size 1 1) (thickness 0.15)) (justify mirror))
     )
@@
     (fp_line (start 0.8 -0.45) (end 0.8 0.45) (layer B.CrtYd) (width 0.05))
     (fp_line (start 0.8 -0.45) (end -0.8 -0.45) (layer B.CrtYd) (width 0.05))
-    (pad 1 smd rect (at -0.45 0 90) (size 0.4 0.6) (layers B.Cu B.Paste B.Mask)
+    (pad 1 smd rect (at -0.45 0) (size 0.4 0.6) (layers B.Cu B.Paste B.Mask)
       (net 1 VBat))
-    (pad 2 smd rect (at 0.45 0 90) (size 0.4 0.6) (layers B.Cu B.Paste B.Mask)
+    (pad 2 smd rect (at 0.45 0) (size 0.4 0.6) (layers B.Cu B.Paste B.Mask)
       (net 5 VBat_Measure))
     (model ${KISYS3DMOD}/Resistors_SMD.3dshapes/R_0402.wrl
@@
   )
   (module Resistors_SMD:R_0402 (layer B.Cu)
-    (at 152.2 96.4 270)
+    (at 153.035 96.52 270)
     (descr "Resistor SMD 0402, reflow soldering, Vishay (see dcrcw.pdf)")
     (tags "resistor 0402")
@@
   (gr_line (start 162.4 97.6) (end 162.4 85.2) (layer Edge.Cuts) (width 0.15))
   (gr_line (start 139.8 97.8) (end 162.4 97.8) (layer Edge.Cuts) (width 0.15))
-  (segment (start 144.5 86.65) (end 145.05 86.65) (width 0.25) (layer B.Cu) (net 1))
-  (segment (start 145.05 86.65) (end 146 85.7) (width 0.25) (layer B.Cu) (net 1))
+  (segment (start 144.5 86.65) (end 145.718 86.65) (width 0.25) (layer B.Cu) (net 1))
+  (segment (start 145.718 86.65) (end 145.796 86.572) (width 0.25) (layer B.Cu) (net 1))
+  (segment (start 147.79 95.15) (end 149.414 96.774) (width 0.25) (layer B.Cu) (net 1))
+  (segment (start 149.414 96.774) (end 150.68 96.774) (width 0.25) (layer B.Cu) (net 1))
+  (segment (start 147.79 93.4) (end 147.79 95.15) (width 0.25) (layer B.Cu) (net 1))
   (segment (start 144.5 86.65) (end 144.75 86.65) (width 0.25) (layer B.Cu) (net 1))
   (segment (start 140.95 93) (end 140.5 93) (width 0.25) (layer B.Cu) (net 1))
@@
   (segment (start 143.4 89.16359) (end 143.4 86.97) (width 0.25) (layer B.Cu) (net 1))
   (segment (start 143.72 86.65) (end 144.5 86.65) (width 0.25) (layer B.Cu) (net 1))
-  (segment (start 150.04 97.4) (end 152.65 97.4) (width 0.25) (layer B.Cu) (net 1))
-  (segment (start 152.65 97.4) (end 153.2 96.85) (width 0.25) (layer B.Cu) (net 1))
-  (segment (start 153.2 96.85) (end 153.3 96.85) (width 0.25) (layer B.Cu) (net 1))
-  (segment (start 147.79 93.4) (end 147.79 95.15) (width 0.25) (layer B.Cu) (net 1))
-  (segment (start 147.79 95.15) (end 150.04 97.4) (width 0.25) (layer B.Cu) (net 1))
   (segment (start 140.95 93) (end 140.95 93.55) (width 0.25) (layer B.Cu) (net 1))
   (segment (start 140.95 93.55) (end 141.2 93.8) (width 0.25) (layer B.Cu) (net 1))
@@
   (segment (start 158.196001 85.424999) (end 145.525001 85.424999) (width 0.25) (layer F.Cu) (net 4))
   (segment (start 159.475001 86.703999) (end 158.196001 85.424999) (width 0.25) (layer F.Cu) (net 4))
+  (segment (start 151.58 96.774) (end 152.284 96.07) (width 0.25) (layer B.Cu) (net 5))
+  (segment (start 152.284 96.07) (end 153.035 96.07) (width 0.25) (layer B.Cu) (net 5))
+  (segment (start 154.35 95.6) (end 153.88 96.07) (width 0.25) (layer B.Cu) (net 5))
+  (segment (start 153.88 96.07) (end 153.035 96.07) (width 0.25) (layer B.Cu) (net 5))
   (segment (start 154.25 96.55) (end 154.25 95.7) (width 0.25) (layer F.Cu) (net 5))
   (segment (start 154.25 95.7) (end 154.35 95.6) (width 0.25) (layer F.Cu) (net 5))
-  (segment (start 153.3 95.95) (end 152.2 95.95) (width 0.25) (layer B.Cu) (net 5))
-  (segment (start 154 95.95) (end 153.3 95.95) (width 0.25) (layer B.Cu) (net 5))
-  (segment (start 154.35 95.6) (end 154 95.95) (width 0.25) (layer B.Cu) (net 5))
   (segment (start 154.2204 95.7296) (end 154.35 95.6) (width 0.25) (layer F.Cu) (net 5))
   (via (at 154.35 95.6) (size 0.6) (drill 0.2) (layers F.Cu B.Cu) (net 5))
