File: _autosave-Duiventrack v1.kicad_pcb (KiCad board)
At the start: 2 copper layers, 22.6 x 12.8 mm, 28 parts, among them P1 CONN_01X07, P2 CONN_01X02, U1 MCP1711-SOT23-5, U2 SP-ABZ-G

Commit message: Small changes
Parts:
- moved R1 2.20 mm to (151.1, 96.8), turned to 0 degrees
- moved C1 0.90 mm to (145.8, 87.1)
- moved R2 0.84 mm to (153.0, 96.5)
Routing:
- net VBat: track 33.0 -> 29.4 mm
- net VBat_Measure: track 3.47 -> 4.05 mm
